File: Hardware/220AC-mini-C3-board/220AC-mini-C3-board.kicad_pcb (KiCad board)
At the start: 2 copper layers, 52.7 x 52.7 mm, 18 parts, among them J1 AC MAINS POWER, J2 ON/OFF switch, J3 Conn_01x04, K1 HF163-F, Q1 Q_NPN_CBE, Q2 Q_NPN_CBE, U1 PBO-3C-3

Commit message: Make revision folders also for production
Parts:
- turned C11 to 90 degrees
Routing:
- net Net-(C1-Pad1): track 11.3 -> 22.2 mm
- net Net-(C1-Pad2): track 21.5 -> 13.0 mm
Changed lines of the file:
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@@
   )
   (footprint "Capacitor_SMD:CP_Elec_10x14.3" (layer "F.Cu")
-    (at 142.56 88.26 -90)
+    (at 142.56 88.26 90)
     (descr "SMD capacitor, aluminum electrolytic, Vishay 1014, 10.0x14.3mm, http://www.vishay.com/docs/28395/150crz.pdf")
     (tags "capacitor electrolytic")
@@
     (property "Sheetname" "")
     (attr smd)
-    (fp_text reference "C11" (at 6.31 2.88 180) (layer "F.SilkS")
+    (fp_text reference "C11" (at 6.31 2.88) (layer "F.SilkS")
       (effects (font (size 1 1) (thickness 0.15)))
     )
@@
     (fp_line (start -5.25 -4.25) (end -5.25 4.25) (layer "F.Fab") (width 0.1))
     (fp_circle (center 0 0) (end 5 0) (layer "F.Fab") (width 0.1) (fill none))
-    (pad "1" smd roundrect (at -4.2 0 270) (size 4.4 2.5) (layers "F.Cu" "F.Paste" "F.Mask") (roundrect_rratio 0.1)
+    (pad "1" smd roundrect (at -4.2 0 90) (size 4.4 2.5) (layers "F.Cu" "F.Paste" "F.Mask") (roundrect_rratio 0.1)
       (net 1 "Net-(C1-Pad1)") (pintype "passive"))
-    (pad "2" smd roundrect (at 4.2 0 270) (size 4.4 2.5) (layers "F.Cu" "F.Paste" "F.Mask") (roundrect_rratio 0.1)
+    (pad "2" smd roundrect (at 4.2 0 90) (size 4.4 2.5) (layers "F.Cu" "F.Paste" "F.Mask") (roundrect_rratio 0.1)
       (net 2 "Net-(C1-Pad2)") (pintype "passive"))
     (model "${KICAD6_3DMODEL_DIR}/Capacitor_SMD.3dshapes/CP_Elec_10x14.3.wrl"
@@
     (effects (font (size 1 1) (thickness 0.15)))
   )
-  (segment (start 143.390001 83.229999) (end 142.56 84.06) (width 1) (layer "F.Cu") (net 1))
-  (segment (start 143.390001 73.14) (end 143.390001 83.229999) (width 1) (layer "F.Cu") (net 1))
+  (segment (start 146.16 78.88) (end 146.16 86.33) (width 1) (layer "F.Cu") (net 1))
+  (segment (start 142.56 89.93) (end 142.56 92.46) (width 1) (layer "F.Cu") (net 1))
+  (segment (start 146.16 86.33) (end 142.56 89.93) (width 1) (layer "F.Cu") (net 1))
+  (segment (start 143.25 75.97) (end 146.16 78.88) (width 1) (layer "F.Cu") (net 1))
+  (segment (start 143.25 72.92) (end 143.25 75.97) (width 1) (layer "F.Cu") (net 1))
   (segment (start 139.390001 73.14) (end 140.300001 74.05) (width 1) (layer "F.Cu") (net 2))
-  (segment (start 140.139473 90.039473) (end 142.56 92.46) (width 1) (layer "F.Cu") (net 2))
   (segment (start 140.300001 74.05) (end 140.3 79.7679) (width 1) (layer "F.Cu") (net 2))
-  (segment (start 140.3 79.7679) (end 138.9679 81.1) (width 1) (layer "F.Cu") (net 2))
-  (segment (start 138.9679 81.1) (end 138.9679 87.211046) (width 1) (layer "F.Cu") (net 2))
-  (arc (start 140.139473 90.039473) (mid 139.272382 88.74178) (end 138.9679 87.211046) (width 1) (layer "F.Cu") (net 2))
+  (segment (start 139.1979 80.87) (end 140.3 79.7679) (width 1) (layer "F.Cu") (net 2))
+  (segment (start 139.65 81.15) (end 142.56 84.06) (width 1) (layer "F.Cu") (net 2))
+  (segment (start 139.1979 81.15) (end 139.1979 80.87) (width 1) (layer "F.Cu") (net 2))
   (segment (start 116.58 73.072323) (end 117.622323 72.03) (width 1) (layer "F.Cu") (net 3))
   (segment (start 127.250002 69.100002) (end 125.9 67.75) (width 1) (layer "F.Cu") (net 3))
