File: Hardware/220AC-mini-C3-board/220AC-mini-C3-board-1.0.kicad_pcb (KiCad board)
At the start: 2 copper layers, 52.7 x 52.7 mm, 18 parts, among them J1 AC MAINS POWER, J2 ON/OFF switch, J3 Conn_01x04, K1 HF163-F, Q1 Q_NPN_CBE, Q2 Q_NPN_CBE, U1 PBO-3C-3

Commit message: cambios CAF
Parts:
- moved J2 37.9 mm to (116.0, 88.2), turned to -90 degrees
- moved J3 35.8 mm to (152.7, 95.0)
- moved R2 28.2 mm to (148.7, 102.6), turned to 0 degrees
- moved R3 28.0 mm to (148.7, 99.6), turned to 0 degrees
- moved D1 15.4 mm to (137.6, 98.5)
- moved Q2 14.6 mm to (140.3, 100.1), turned to 0 degrees
- moved Q1 14.2 mm to (140.3, 106.0), turned to 0 degrees
- moved K1 7.53 mm to (130.5, 98.1), turned to 90 degrees
- moved D2 0.40 mm to (123.4, 98.5), turned to -90 degrees
Routing:
- net GND: track 37.4 -> 12.6 mm
- net +3V3: track 47.3 -> 71.8 mm
- net Net-(D2-Pad2): track 11.6 -> 28.7 mm
- net /AC (N): track 17.0 -> 27.6 mm
- net Net-(J2-Pad1): track 13.6 -> 22.3 mm
- net Net-(R1-Pad2): track 0.00 -> 6.21 mm
- net Net-(D1-Pad2): track 21.6 -> 18.7 mm, vias 0 -> 2
- net Net-(Q2-Pad2): track 5.33 -> 6.93 mm
- net /IO_2: track 4.01 -> 3.11 mm
- net /IO_3: track 4.01 -> 3.29 mm
- net Net-(Q1-Pad2): track 11.1 -> 11.8 mm
- net Net-(F1-Pad2): track 6.98 -> 7.58 mm
Other:
- board text added: "V 1.1"
