File: Hardware/S3-27-epaper-touch-pro/S3-27-epaper-touch.kicad_sch (KiCad schematic)
At the start: 61 parts, among them J1 AFC24-S24FIC-00, J2 USB_C_Programming, J3 Conn_01x06, J4 Conn_01x06_Female, J5 Groove sensor, J6 Conn_01x06, Q1 Si1308, Q2 BC817, Q3 BC817, U1 ESP32-S3-WROOM-1-N8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

Commit message: Clear DRC errors
Connections:
- net IO4_ADC1_CH3: now also J3.5 (Pin_5)
- net IO_8: no longer names the net of U1.12 (IO8)
- net IO_8: no longer J3.5 (Pin_5)
- no-connect marks 39 -> 40
Changed lines of the file:
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@@
   (no_connect (at 345.44 86.36))
   (no_connect (at 302.26 48.26))
+  (no_connect (at 161.29 82.55))
   (no_connect (at 292.1 101.6))
   (no_connect (at 201.93 180.34))
@@
     (stroke (width 0) (type default) (color 0 0 0 0))
   )
-  (wire (pts (xy 181.61 140.97) (xy 187.96 140.97))
+  (wire (pts (xy 175.26 140.97) (xy 187.96 140.97))
     (stroke (width 0) (type default) (color 0 0 0 0))
   )
@@
     (effects (font (size 1 1)) (justify left bottom))
   )
-  (text "5V IN" (at 173.99 139.7 0)
+  (text "5V IN" (at 167.64 139.7 0)
     (effects (font (size 1.27 1.27)) (justify left bottom))
   )
@@
     (effects (font (size 1.27 1.27)) (justify right bottom))
   )
+  (label "IO4_ADC1_CH3" (at 187.96 138.43 180)
+    (effects (font (size 1.27 1.27)) (justify right bottom))
+  )
   (label "ENABLE" (at 140.97 59.69 180)
     (effects (font (size 1.27 1.27)) (justify right bottom))
@@
     (effects (font (size 1.27 1.27)) (justify left bottom))
   )
-  (label "IO_8" (at 187.96 138.43 180)
-    (effects (font (size 1.27 1.27)) (justify right bottom))
-  )
   (label "IO_18" (at 264.16 140.97 180)
     (effects (font (size 1.27 1.27)) (justify right bottom))
@@
     (effects (font (size 1.27 1.27)) (justify left bottom))
   )
-  (label "IO_8" (at 161.29 82.55 180)
-    (effects (font (size 1.27 1.27)) (justify right bottom))
-  )
   (label "TOUCH_INT" (at 189.23 177.8 180)
     (effects (font (size 1.27 1.27)) (justify right bottom))
@@
     (effects (font (size 1.27 1.27)) (justify right bottom))
   )
-  (global_label "VBUS" (shape input) (at 181.61 140.97 180) (fields_autoplaced)
+  (global_label "VBUS" (shape input) (at 175.26 140.97 180) (fields_autoplaced)
     (effects (font (size 1.27 1.27)) (justify right))
-    (property "Intersheet References" "${INTERSHEET_REFS}" (id 0) (at 174.2983 140.8906 0)
+    (property "Intersheet References" "${INTERSHEET_REFS}" (id 0) (at 167.9483 140.8906 0)
       (effects (font (size 1.27 1.27)) (justify right) hide)
     )

Commit message: S3: Do not use MOSI in JTAG data pins
Connections:
- net 3231_INT: now also U1.12 (IO8); no longer U1.21 (IO13)
- net EPD_MOSI: now also U1.21 (IO13); no longer U1.14 (IO20)
Other:
- note added: "JTAG D+"
- note added: "JTAG D-"
Changed lines of the file:
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@@
   (no_connect (at 345.44 86.36))
   (no_connect (at 302.26 48.26))
-  (no_connect (at 161.29 82.55))
   (no_connect (at 292.1 101.6))
   (no_connect (at 201.93 180.34))
   (no_connect (at 201.93 87.63))
   (no_connect (at 276.86 83.82))
+  (no_connect (at 161.29 87.63))
   (polyline (pts (xy 372.11 118.11) (xy 372.11 151.13))
     (stroke (width 0) (type default) (color 0 0 0 0))
@@
   )
   (wire (pts (xy 160.02 97.79) (xy 161.29 97.79))
-    (stroke (width 0) (type default) (color 0 0 0 0))
-  )
-  (wire (pts (xy 160.02 87.63) (xy 161.29 87.63))
     (stroke (width 0) (type default) (color 0 0 0 0))
   )
@@
     (effects (font (size 1.27 1.27)) (justify left bottom))
   )
+  (text "JTAG D+" (at 152.4 87.63 0)
+    (effects (font (size 1.27 1.27)) (justify left bottom))
+  )
   (text "RESET" (at 172.72 60.96 0)
     (effects (font (size 1.27 1.27)) (justify left bottom))
@@
     (effects (font (size 5 5)) (justify left bottom))
   )
+  (text "JTAG D-" (at 152.4 85.09 0)
+    (effects (font (size 1.27 1.27)) (justify left bottom))
+  )
   (text "Mounting w/ wall switch" (at 299.72 160.02 0)
     (effects (font (size 1.27 1.27)) (justify left bottom))
@@
     (effects (font (size 1.27 1.27)) (justify right bottom))
   )
-  (label "3231_INT" (at 203.2 105.41 0)
-    (effects (font (size 1.27 1.27)) (justify left bottom))
+  (label "3231_INT" (at 161.29 82.55 180)
+    (effects (font (size 1.27 1.27)) (justify right bottom))
   )
   (label "IO_18" (at 264.16 140.97 180)
@@
     (effects (font (size 1.27 1.27)) (justify right bottom))
   )
-  (label "EPD_MOSI" (at 160.02 87.63 180)
-    (effects (font (size 1.27 1.27)) (justify right bottom))
-  )
   (label "IO_2" (at 204.47 62.23 0)
     (effects (font (size 1.27 1.27)) (justify left bottom))
@@
     (effects (font (size 1.27 1.27)) (justify left bottom))
   )
+  (label "EPD_MOSI" (at 203.2 105.41 0)
+    (effects (font (size 1.27 1.27)) (justify left bottom))
+  )

Commit message: Add files via upload
Changes
R16 0R = IO46 Resistor for Compatibility to ESP32 WROOM
R15 changed package to 0603(was 0402)
Fixed Layout error at R15
Rerouted RTS Line to enable 2 Layer Board
Rerouted 3.3V next to J3
Changed orientation of C3
Routed IO18 to J7 to make space for USB Host
Added USB Port J7

TODO:
Need to double check usage of ESP32 Wroom if they are compatible to current pinning
(NOT with current pinning)
Parts:
- added J7: Conn_01x03, Connector_PinSocket_2.54mm:PinSocket_1x03_P2.54mm_Vertical, symbol Connector_Generic:Conn_01x03
- added R16: 0R, Resistor_SMD:R_0603_1608Metric, symbol Device:R_Small
- R15: footprint Resistor_SMD:R_0402_1005Metric -> Resistor_SMD:R_0603_1608Metric; LCSC C137974 -> (none)
Connections:
- net GND: now also R16.1
- net IO_18: now also J7.3 (Pin_3); no longer J6.6 (Pin_6)
- net USB_D-: now reaches U1.13 (IO19)
- net USB_D-: now also J7.2 (Pin_2)
- net USB_D+: now reaches U1.14 (IO20)
- net USB_D+: now also J7.1 (Pin_1)
- net at U1.16 (IO46): now also R16.2
- no-connect marks 40 -> 38
Other:
- note added: "Changes R16 0R = IO46 Resistor for Compatibility to ESP32 WROOM R15 changed package to 0603(was 0402) Fixed Layout error at R15 Rerouted RTS Line to enable 2 Layer Board Rerouted 3.3V next to J3 Changed orientation of C3 Routed IO18 to J7 to make space for USB Host Added USB Port J7 TODO: Need to double check usage of ESP32 Wroom if they are compatible to current pinning (NOT with current pinning)"
- note added: "USB-JTAG signals (if CP2102 is not OK)"
- note removed: "JTAG D+"
- note removed: "JTAG D-"
