File: Hardware/C3-27-epaper-touch/C3-27-epaper-touch.kicad_pcb (KiCad board)
At the start: 4 copper layers, 70.2 x 71 mm, 62 parts, among them J1 AFC24-S24FIC-00, J2 USB_C_Programming, J3 Conn_01x06, J4 Conn_01x06_Female, J5 Groove sensor, Q1 Si1308, Q2 BC817, Q3 BC817, U1 ESP32-C3-WROOM-02-N4, U2 CP2102N-A02-GQFN28R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

Commit message: C3 Rev 1.1 tests
Routing:
- net /TOUCH_SCL: track 85.4 -> 86.3 mm
Changed lines of the file:
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@@
   (segment (start 138.85 78.175) (end 141.575 78.175) (width 0.25) (layer "F.Cu") (net 7))
   (segment (start 141.575 78.175) (end 142.100001 78.700001) (width 0.25) (layer "F.Cu") (net 7))
-  (segment (start 128.93 82.18) (end 128.93 84.45) (width 0.25) (layer "F.Cu") (net 8))
+  (segment (start 126.971501 73.878499) (end 124.375 76.475) (width 0.25) (layer "F.Cu") (net 8))
   (segment (start 120.150001 80.699999) (end 120.150001 90.139) (width 0.25) (layer "F.Cu") (net 8))
   (segment (start 120.150001 90.439) (end 120.150001 93.150001) (width 0.25) (layer "F.Cu") (net 8))
-  (segment (start 128.93 84.45) (end 130.105 85.625) (width 0.25) (layer "F.Cu") (net 8))
   (segment (start 150.115085 114.655085) (end 148.66 113.2) (width 0.25) (layer "F.Cu") (net 8))
+  (segment (start 127.59 81.95) (end 125.19 81.95) (width 0.25) (layer "F.Cu") (net 8))
   (segment (start 151.264 114.655085) (end 150.115085 114.655085) (width 0.25) (layer "F.Cu") (net 8))
-  (segment (start 122.59 78.26) (end 122.5 78.35) (width 0.25) (layer "F.Cu") (net 8))
+  (segment (start 124.375 81.135) (end 124.375 76.475) (width 0.25) (layer "F.Cu") (net 8))
+  (segment (start 130.105 85.625) (end 128.93 84.45) (width 0.25) (layer "F.Cu") (net 8))
   (segment (start 148.37 112.91) (end 146.59 112.91) (width 0.25) (layer "F.Cu") (net 8))
-  (segment (start 130.105 85.625) (end 131.135 85.625) (width 0.25) (layer "F.Cu") (net 8))
   (segment (start 121.04 94.04) (end 120.85 93.85) (width 0.25) (layer "F.Cu") (net 8))
   (segment (start 151.264 114.655085) (end 154.630085 114.655085) (width 0.25) (layer "F.Cu") (net 8))
-  (segment (start 126.971501 73.878499) (end 122.5 78.35) (width 0.25) (layer "F.Cu") (net 8))
+  (segment (start 128.93 84.45) (end 128.93 83.29) (width 0.25) (layer "F.Cu") (net 8))
   (segment (start 148.66 113.2) (end 148.37 112.91) (width 0.25) (layer "F.Cu") (net 8))
-  (segment (start 128.93 82.18) (end 125.01 78.26) (width 0.25) (layer "F.Cu") (net 8))
+  (segment (start 125.19 81.95) (end 124.375 81.135) (width 0.25) (layer "F.Cu") (net 8))
   (segment (start 121.05 94.05) (end 120.85 93.85) (width 0.25) (layer "F.Cu") (net 8))
-  (segment (start 125.01 78.26) (end 122.59 78.26) (width 0.25) (layer "F.Cu") (net 8))
+  (segment (start 128.93 83.29) (end 127.59 81.95) (width 0.25) (layer "F.Cu") (net 8))
   (segment (start 121.04 99.4) (end 121.04 94.04) (width 0.25) (layer "F.Cu") (net 8))
+  (segment (start 131.135 85.625) (end 130.105 85.625) (width 0.25) (layer "F.Cu") (net 8))
   (segment (start 154.630085 114.655085) (end 155 115.025) (width 0.25) (layer "F.Cu") (net 8))
+  (segment (start 124.375 76.475) (end 122.5 78.35) (width 0.25) (layer "F.Cu") (net 8))
   (segment (start 122.5 78.35) (end 120.150001 80.699999) (width 0.25) (layer "F.Cu") (net 8))
   (segment (start 126.971501 72.2) (end 126.971501 73.878499) (width 0.25) (layer "F.Cu") (net 8))

Commit message: 1.2 is ready, this time MCU can be soldered already
Parts:
- R12: value 10 K -> 4.7K
Changed lines of the file:
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@@
   )
   (paper "A4")
+  (title_block
+    (title "C3 epaper controller w/touch")
+    (date "2023-03-15")
+    (rev "1.2")
+    (company "FASANI CORPORATION")
+  )
   (layers
     (0 "F.Cu" signal)
@@
     (descr "Resistor SMD 0603 (1608 Metric), square (rectangular) end terminal, IPC_7351 nominal, (Body size source: IPC-SM-782 page 72, https://www.pcb-3d.com/wordpress/wp-content/uploads/ipc-sm-782a_amendment_1_and_2.pdf), generated with kicad-footprint-generator")
     (tags "resistor")
-    (property "LCSC" "C25804")
+    (property "LCSC" "C23162")
     (property "Sheetfile" "C3-27-epaper-touch.kicad_sch")
     (property "Sheetname" "")
@@
       (effects (font (size 0.7 0.7) (thickness 0.13)))
     )
-    (fp_text value "10 K" (at 0 1.43 90) (layer "F.Fab")
-      (effects (font (size 1 1) (thickness 0.15)))
-    )
+    (fp_text value "4.7K" (at 0 1.43 90) (layer "F.Fab")
+      (effects (font (size 1 1) (thickness 0.15)))
+    )
