File: Hardware/C3-27-epaper-touch/C3-27-epaper-touch.kicad_sch (KiCad schematic)
At the start: 62 parts, among them J1 AFC24-S24FIC-00, J2 USB_C_Programming, J3 Conn_01x06, J4 Conn_01x06_Female, J5 Groove sensor, Q1 Si1308, Q2 BC817, Q3 BC817, U1 ESP32-C3-WROOM-02-N4, U2 CP2102N-A02-GQFN28R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

Commit message: Update C15 put it closer to LDO
Parts:
- D5: Height 1.22 -> (none); LCSC (none) -> C3040626
- U4: LCSC (none) -> C7440
Changed lines of the file:
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@@
+      (effects (font (size 1.27 1.27)) hide)
+    )
+    (property "LCSC" "C7440" (id 4) (at 91.44 194.31 0)
       (effects (font (size 1.27 1.27)) hide)
     )
@@
       (effects (font (size 1.27 1.27)) (justify left) hide)
     )
-    (property "Datasheet" "https://nl.mouser.com/datasheet/2/240/Littelfuse_TVS_Diode_Array_SP05_Datasheet.pdf-777043.pdf" (id 3) (at 335.28 85.09 0)
+    (property "Datasheet" "https://jlcpcb.com/partdetail/TechPublic-SP0503BAHTG/C3040626" (id 3) (at 335.28 85.09 0)
       (effects (font (size 1.27 1.27)) (justify left) hide)
     )
@@
       (effects (font (size 1.27 1.27)) (justify left) hide)
     )
-    (property "Height" "1.22" (id 5) (at 340.36 85.09 0)
-      (effects (font (size 1.27 1.27)) (justify left) hide)
-    )
+    (property "LCSC" "C3040626" (id 5) (at 340.36 85.09 0)
+      (effects (font (size 1.27 1.27)) (justify left) hide)
+    )

Commit message: Mark properly D+ & D- lines
Connections:
- net D+: now reaches D5.3 (K_2), J2.A6 (D+), J2.B6 (D+), U2.4 (D+)
- net D-: now reaches D5.4 (K_3), J2.A7 (D-), J2.B7 (D-), U2.5 (D-)
Changed lines of the file:
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@@
     (effects (font (size 1.27 1.27)) (justify left bottom))
+  )
+  (label "D+" (at 344.17 76.2 270)
+    (effects (font (size 1.27 1.27)) (justify right bottom))
   )
   (label "IO_2" (at 203.2 90.17 0)
@@
     (effects (font (size 1.27 1.27)) (justify left bottom))
   )
+  (label "D-" (at 344.17 73.66 90)
+    (effects (font (size 1.27 1.27)) (justify left bottom))
+  )

Commit message: Update 1.1 R14 & R15 VUSB sense CP2102
Parts:
- R15: footprint Resistor_SMD:R_0402_1005Metric -> Resistor_SMD:R_0603_1608Metric; LCSC C137974 -> C137715
Changed lines of the file:
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@@
       (effects (font (size 1.27 1.27)) (justify left))
     )
-    (property "Footprint" "Resistor_SMD:R_0402_1005Metric" (id 2) (at 313.69 41.91 0)
-      (effects (font (size 1.27 1.27)) hide)
-    )
-    (property "Datasheet" "https://jlcpcb.com/partdetail/Yageo-RC0402FR0747K5L/C137974" (id 3) (at 313.69 41.91 0)
-      (effects (font (size 1.27 1.27)) hide)
-    )
-    (property "LCSC" "C137974" (id 4) (at 313.69 41.91 90)
+    (property "Footprint" "Resistor_SMD:R_0603_1608Metric" (id 2) (at 313.69 41.91 0)
+      (effects (font (size 1.27 1.27)) hide)
+    )
+    (property "Datasheet" "https://jlcpcb.com/partdetail/Yageo-RC0603FR0747K5L/C137715" (id 3) (at 313.69 41.91 0)
+      (effects (font (size 1.27 1.27)) hide)
+    )
+    (property "LCSC" "C137715" (id 4) (at 313.69 41.91 90)
       (effects (font (size 1.27 1.27)) hide)
     )
@@
     )
     (path "/f03960ef-9e49-45d2-a9fd-2f2de73439b2"
-      (reference "R15") (unit 1) (value "47K") (footprint "Resistor_SMD:R_0402_1005Metric")
+      (reference "R15") (unit 1) (value "47K") (footprint "Resistor_SMD:R_0603_1608Metric")
     )
     (path "/21439738-76b8-4267-91fd-2ea304ae429f"

Commit message: C3 1.1 replace C13 to be 4.7uF
Parts:
- C13: value 100nF -> 4.7uF; LCSC C28233 -> C1779
Changed lines of the file:
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@@
       (effects (font (size 1.27 1.27)) (justify right))
     )
-    (property "Value" "100nF" (id 1) (at 327.66 64.77 90)
+    (property "Value" "4.7uF" (id 1) (at 327.66 64.77 90)
       (effects (font (size 1.27 1.27)) (justify right))
     )
@@
       (effects (font (size 1.27 1.27)) hide)
     )
-    (property "LCSC" "C28233" (id 4) (at 330.2 68.58 0)
+    (property "LCSC" "C1779" (id 4) (at 330.2 68.58 0)
       (effects (font (size 1.27 1.27)) hide)
     )
@@
     )
     (path "/e010b6fb-2fb9-4bfd-b982-6a597128c5da"
-      (reference "C13") (unit 1) (value "100nF") (footprint "Capacitor_SMD:C_0805_2012Metric")
+      (reference "C13") (unit 1) (value "4.7uF") (footprint "Capacitor_SMD:C_0805_2012Metric")
     )
     (path "/858e1609-0117-4a64-a4cb-af2f22b2944b"

Commit message: 1.2 is ready, this time MCU can be soldered already
Parts:
- R12: value 10 K -> 4.7K; LCSC C25804 -> C23162
Other:
- note added: "REV DESCRIPTION 1.2 R12 RTC interrupt pull-up now changed to 4K7 1.1 C3 working PCB only one issue found: RTC INT pull-up 10K is reporting always LOW 1.0 Initial version with many Harware errors (MOSI routed to IO9, that needs to be pull-up in BOOT)"
- note added: "Revision LOGs"
- moved on the sheet: J5
Changed lines of the file:
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@@
     (title "ESP32-C3 epaper controller with touch")
     (date "2022-11-22")
-    (rev "1.1")
+    (rev "1.2")
     (comment 1 "be used in home appliances with no more than 200 Watts top consumption.")
     (comment 2 "industrial heavy load devices. This an experimental switch that should only")
@@
     (stroke (width 0) (type default) (color 0 0 0 0))
   )
-  (polyline (pts (xy 220.98 217.17) (xy 203.2 217.17))
+  (polyline (pts (xy 220.98 207.01) (xy 203.2 207.01))
     (stroke (width 0) (type default) (color 0 0 0 0))
   )
@@
     (stroke (width 0) (type default) (color 0 0 0 0))
   )
+  (polyline (pts (xy 240.03 160.02) (xy 297.18 160.02))
+    (stroke (width 0) (type default) (color 0 0 0 0))
+  )
   (wire (pts (xy 189.23 177.8) (xy 193.04 177.8))
     (stroke (width 0) (type default) (color 0 0 0 0))
@@
     (stroke (width 0) (type default) (color 0 0 0 0))
   )
+  (polyline (pts (xy 240.03 203.2) (xy 401.32 203.2))
+    (stroke (width 0) (type default) (color 0 0 0 0))
+  )
   (wire (pts (xy 63.5 175.26) (xy 63.5 179.07))
     (stroke (width 0) (type default) (color 0 0 0 0))
@@
     (stroke (width 0) (type default) (color 0 0 0 0))
   )
-  (polyline (pts (xy 149.86 251.46) (xy 220.98 251.46))
+  (polyline (pts (xy 149.86 241.3) (xy 220.98 241.3))
     (stroke (width 0) (type default) (color 0 0 0 0))
   )
@@
     (stroke (width 0) (type default) (color 0 0 0 0))
   )
-  (polyline (pts (xy 165.1 217.17) (xy 149.86 217.17))
+  (polyline (pts (xy 165.1 207.01) (xy 149.86 207.01))
     (stroke (width 0) (type default) (color 0 0 0 0))
   )
@@
     (stroke (width 0) (type default) (color 0 0 0 0))
   )
-  (polyline (pts (xy 149.86 217.17) (xy 149.86 251.46))
+  (polyline (pts (xy 149.86 207.01) (xy 149.86 241.3))
     (stroke (width 0) (type default) (color 0 0 0 0))
   )
@@
     (stroke (width 0) (type default) (color 0 0 0 0))
   )
+  (polyline (pts (xy 336.55 160.02) (xy 401.32 160.02))
+    (stroke (width 0) (type default) (color 0 0 0 0))
+  )
   (polyline (pts (xy 292.1 134.62) (xy 292.1 148.59))
     (stroke (width 0) (type default) (color 0 0 0 0))
@@
     (stroke (width 0) (type default) (color 0 0 0 0))
   )
-  (wire (pts (xy 186.69 238.76) (xy 200.66 238.76))
+  (wire (pts (xy 186.69 228.6) (xy 200.66 228.6))
     (stroke (width 0) (type default) (color 0 0 0 0))
   )
@@
     (stroke (width 0) (type default) (color 0 0 0 0))
   )
+  (polyline (pts (xy 240.03 160.02) (xy 240.03 203.2))
+    (stroke (width 0) (type default) (color 0 0 0 0))
+  )
   (wire (pts (xy 205.74 64.77) (xy 203.2 64.77))
     (stroke (width 0) (type default) (color 0 0 0 0))
@@
     (stroke (width 0) (type default) (color 0 0 0 0))
   )
+  (polyline (pts (xy 401.32 203.2) (xy 401.32 160.02))
+    (stroke (width 0) (type default) (color 0 0 0 0))
+  )
   (wire (pts (xy 101.6 113.03) (xy 101.6 110.49))
     (stroke (width 0) (type default) (color 0 0 0 0))
@@
     (stroke (width 0) (type default) (color 0 0 0 0))
   )
-  (wire (pts (xy 200.66 241.3) (xy 186.69 241.3))
+  (wire (pts (xy 200.66 231.14) (xy 186.69 231.14))
     (stroke (width 0) (type default) (color 0 0 0 0))
   )
@@
     (stroke (width 0) (type default) (color 0 0 0 0))
   )
-  (polyline (pts (xy 220.98 251.46) (xy 220.98 217.17))
+  (polyline (pts (xy 220.98 241.3) (xy 220.98 207.01))
     (stroke (width 0) (type default) (color 0 0 0 0))
   )
@@
     (effects (font (size 1.27 1.27)) (justify left bottom))
   )
-  (text "Groove I2C connector" (at 167.64 218.44 0)
+  (text "REV DESCRIPTION\n1.2 R12 RTC interrupt pull-up now changed to 4K7\n1.1 C3 working PCB only one issue found: RTC INT pull-up 10K is reporting always LOW\n1.0 Initial version with many Harware errors (MOSI routed to IO9, that needs to be pull-up in BOOT)"
+    (at 242.57 175.26 0)
+    (effects (font (size 2 2)) (justify left bottom))
+  )
+  (text "Groove I2C connector" (at 167.64 208.28 0)
+    (effects (font (size 2 2)) (justify left bottom))
+  )
+  (text "Revision LOGs" (at 307.34 161.29 0)
     (effects (font (size 2 2)) (justify left bottom))
   )
@@
     (effects (font (size 1.27 1.27)) (justify left bottom))
   )
-  (label "TOUCH_SCL" (at 186.69 233.68 0)
+  (label "TOUCH_SCL" (at 186.69 223.52 0)
     (effects (font (size 1.27 1.27)) (justify left bottom))
   )
@@
     (effects (font (size 1.27 1.27)) (justify right bottom))
   )
-  (label "TOUCH_SDA" (at 186.69 236.22 0)
+  (label "TOUCH_SDA" (at 186.69 226.06 0)
     (effects (font (size 1.27 1.27)) (justify left bottom))
   )
@@
     (pin "2")
   )
-  (symbol (lib_id "MOLEX-I2C-532530470:532530470") (at 186.69 233.68 0) (mirror y) (unit 1)
+  (symbol (lib_id "MOLEX-I2C-532530470:532530470") (at 186.69 223.52 0) (mirror y) (unit 1)
     (in_bom yes) (on_board yes)
-    (property "Reference" "J5" (id 0) (at 177.8 226.9924 0)
+    (property "Reference" "J5" (id 0) (at 177.8 216.8324 0)
       (effects (font (size 1.524 1.524)))
     )
-    (property "Value" "Groove sensor" (id 1) (at 180.34 229.87 0)
+    (property "Value" "Groove sensor" (id 1) (at 180.34 219.71 0)
       (effects (font (size 1.524 1.524)))
     )
-    (property "Footprint" "footprint:MOLEX-I2C-532530470" (id 2) (at 176.53 240.284 0)
+    (property "Footprint" "footprint:MOLEX-I2C-532530470" (id 2) (at 176.53 230.124 0)
       (effects (font (size 1.524 1.524)) hide)
     )
-    (property "Datasheet" "" (id 3) (at 186.69 233.68 0)
+    (property "Datasheet" "" (id 3) (at 186.69 223.52 0)
       (effects (font (size 1.524 1.524)))
     )
@@
     (pin "2")
   )
-  (symbol (lib_id "power:+3V3") (at 200.66 238.76 0) (unit 1)
+  (symbol (lib_id "power:+3V3") (at 200.66 228.6 0) (unit 1)
     (in_bom yes) (on_board yes) (fields_autoplaced)
-    (property "Reference" "#PWR017" (id 0) (at 200.66 242.57 0)
+    (property "Reference" "#PWR017" (id 0) (at 200.66 232.41 0)
       (effects (font (size 1.27 1.27)) hide)
     )
-    (property "Value" "+3V3" (id 1) (at 200.66 235.1842 0))
-    (property "Footprint" "" (id 2) (at 200.66 238.76 0)
+    (property "Value" "+3V3" (id 1) (at 200.66 225.0242 0))
+    (property "Footprint" "" (id 2) (at 200.66 228.6 0)
       (effects (font (size 1.27 1.27)) hide)
     )
-    (property "Datasheet" "" (id 3) (at 200.66 238.76 0)
+    (property "Datasheet" "" (id 3) (at 200.66 228.6 0)
       (effects (font (size 1.27 1.27)) hide)
     )
@@
       (effects (font (size 1.27 1.27)) (justify left))
     )
-    (property "Value" "10 K" (id 1) (at 125.9586 196.0122 0)
+    (property "Value" "4.7K" (id 1) (at 125.9586 196.0122 0)
       (effects (font (size 1.27 1.27)) (justify left))
     )
@@
       (effects (font (size 1.27 1.27)) hide)
     )
-    (property "Datasheet" "https://datasheet.lcsc.com/lcsc/2206010045_UNI-ROYAL-Uniroyal-Elec-0603WAF1002T5E_C25804.pdf" (id 3) (at 124.46 194.31 0)
+    (property "Datasheet" "https://jlcpcb.com/partdetail/23889-0603WAF4701T5E/C23162" (id 3) (at 124.46 194.31 0)
       (effects (font (size 1.27 1.27)) hide)
     )
-    (property "LCSC" "C25804" (id 4) (at 124.46 194.31 0)
+    (property "LCSC" "C23162" (id 4) (at 124.46 194.31 0)
       (effects (font (size 1.27 1.27)) hide)
     )
@@
     (pin "1")
   )
-  (symbol (lib_id "power:GND") (at 200.66 241.3 0) (unit 1)
+  (symbol (lib_id "power:GND") (at 200.66 231.14 0) (unit 1)
     (in_bom yes) (on_board yes) (fields_autoplaced)
-    (property "Reference" "#PWR018" (id 0) (at 200.66 247.65 0)
+    (property "Reference" "#PWR018" (id 0) (at 200.66 237.49 0)
       (effects (font (size 1.27 1.27)) hide)
     )
-    (property "Value" "GND" (id 1) (at 200.66 245.7434 0))
-    (property "Footprint" "" (id 2) (at 200.66 241.3 0)
+    (property "Value" "GND" (id 1) (at 200.66 235.5834 0))
+    (property "Footprint" "" (id 2) (at 200.66 231.14 0)
       (effects (font (size 1.27 1.27)) hide)
     )
-    (property "Datasheet" "" (id 3) (at 200.66 241.3 0)
+    (property "Datasheet" "" (id 3) (at 200.66 231.14 0)
       (effects (font (size 1.27 1.27)) hide)
     )
@@
     )
     (path "/965882ad-ba10-4813-8e31-868947a9b01b"
-      (reference "R12") (unit 1) (value "10 K") (footprint "Resistor_SMD:R_0603_1608Metric")
+      (reference "R12") (unit 1) (value "4.7K") (footprint "Resistor_SMD:R_0603_1608Metric")
     )
     (path "/0e7c6e7a-9a40-4afd-9227-b71859efc35b"

Commit message: C3 PCB add R16 current limiting for RTC backup CAPs
Parts:
- added R16: 22Ω, Resistor_SMD:R_0603_1608Metric, symbol Device:R
Connections:
- net at C17.1, C18.1: now also R16.1; no longer D4.1 (K), U4.8 (VDD)
- new net: D4.1 (K), R16.2, U4.8 (VDD)
Changed lines of the file:
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@@
   (junction (at 69.85 199.39) (diameter 0) (color 0 0 0 0)
   )
+  (junction (at 87.63 175.26) (diameter 0) (color 0 0 0 0)
+  )
   (junction (at 109.22 125.73) (diameter 0) (color 0 0 0 0)
   )
@@
   (junction (at 203.2 77.47) (diameter 0) (color 0 0 0 0)
   )
-  (junction (at 87.63 175.26) (diameter 0) (color 0 0 0 0)
-  )
   (junction (at 168.91 185.42) (diameter 0) (color 0 0 0 0)
   )
@@
     (stroke (width 0) (type default) (color 0 0 0 0))
   )
-  (wire (pts (xy 87.63 175.26) (xy 63.5 175.26))
-    (stroke (width 0) (type default) (color 0 0 0 0))
-  )
   (wire (pts (xy 80.01 77.47) (xy 78.74 77.47))
     (stroke (width 0) (type default) (color 0 0 0 0))
@@
     (stroke (width 0) (type default) (color 0 0 0 0))
   )
+  (wire (pts (xy 71.12 175.26) (xy 87.63 175.26))
+    (stroke (width 0) (type default) (color 0 0 0 0))
+  )
   (wire (pts (xy 77.47 199.39) (xy 78.74 199.39))
     (stroke (width 0) (type default) (color 0 0 0 0))
@@
     (stroke (width 0) (type default) (color 0 0 0 0))
   )
-  (wire (pts (xy 99.06 173.99) (xy 99.06 175.26))
-    (stroke (width 0) (type default) (color 0 0 0 0))
-  )
   (wire (pts (xy 101.6 196.85) (xy 118.11 196.85))
     (stroke (width 0) (type default) (color 0 0 0 0))
@@
     (stroke (width 0) (type default) (color 0 0 0 0))
   )
+  (wire (pts (xy 99.06 175.26) (xy 111.76 175.26))
+    (stroke (width 0) (type default) (color 0 0 0 0))
+  )
   (polyline (pts (xy 220.98 160.02) (xy 220.98 203.2))
     (stroke (width 0) (type default) (color 0 0 0 0))
@@
     (pin "1")
   )
+  (symbol (lib_id "Device:R") (at 67.31 175.26 90) (unit 1)
+    (in_bom yes) (on_board yes)
+    (property "Reference" "R16" (id 0) (at 66.04 172.72 90))
+    (property "Value" "22Ω" (id 1) (at 67.31 177.8 90))
+    (property "Footprint" "Resistor_SMD:R_0603_1608Metric" (id 2) (at 67.31 177.038 90)
+      (effects (font (size 1.27 1.27)) hide)
+    )
+    (property "Datasheet" "https://jlcpcb.com/partdetail/188958-RCT0322R1FLF/C177566" (id 3) (at 67.31 175.26 0)
+      (effects (font (size 1.27 1.27)) hide)
+    )
+    (property "LCSC" "C177566" (id 4) (at 67.31 175.26 90)
+      (effects (font (size 1.27 1.27)) hide)
+    )
+    (pin "1")
+    (pin "2")
+  )
   (symbol (lib_id "power:GND") (at 332.74 49.53 0) (unit 1)
     (in_bom yes) (on_board yes)
@@
   (symbol (lib_id "Diode:MBR0530") (at 95.25 175.26 0) (unit 1)
     (in_bom yes) (on_board yes)
-    (property "Reference" "D4" (id 0) (at 95.25 171.45 0))
+    (property "Reference" "D4" (id 0) (at 95.25 172.72 0))
     (property "Value" "1N5819WS" (id 1) (at 92.71 179.07 0)
       (effects (font (size 1.27 1.27)) hide)
@@
     (pin "2")
   )
-  (symbol (lib_id "power:+3.3V") (at 99.06 173.99 0) (unit 1)
+  (symbol (lib_id "power:+3.3V") (at 111.76 175.26 0) (unit 1)
     (in_bom yes) (on_board yes)
-    (property "Reference" "#PWR014" (id 0) (at 99.06 177.8 0)
+    (property "Reference" "#PWR014" (id 0) (at 111.76 179.07 0)
       (effects (font (size 1.27 1.27)) hide)
     )
-    (property "Value" "+3.3V" (id 1) (at 101.6 173.99 0))
-    (property "Footprint" "" (id 2) (at 99.06 173.99 0)
+    (property "Value" "+3.3V" (id 1) (at 114.3 175.26 0))
+    (property "Footprint" "" (id 2) (at 111.76 175.26 0)
       (effects (font (size 1.27 1.27)) hide)
     )
-    (property "Datasheet" "" (id 3) (at 99.06 173.99 0)
+    (property "Datasheet" "" (id 3) (at 111.76 175.26 0)
       (effects (font (size 1.27 1.27)) hide)
     )
@@
       (reference "R15") (unit 1) (value "47K") (footprint "Resistor_SMD:R_0603_1608Metric")
     )
+    (path "/6d704ead-f7d9-4fa5-8510-b2eda0f5facb"
+      (reference "R16") (unit 1) (value "22Ω") (footprint "Resistor_SMD:R_0603_1608Metric")
+    )
     (path "/21439738-76b8-4267-91fd-2ea304ae429f"

Commit message: Update schematics. Introduce Rev log
Other:
- note added: "REV DESCRIPTION 1.2 R12 RTC interrupt pull-up now changed to 4K7 Added R16 22Ω currrent limiter to charge RTC backup capacitors 1.1 C3 working PCB only one issue found: RTC INT pull-up 10K is reporting always LOW 1.0 Initial version with many Harware errors (MOSI routed to IO9, that needs to be pull-up in BOOT)"
- note removed: "REV DESCRIPTION 1.2 R12 RTC interrupt pull-up now changed to 4K7 1.1 C3 working PCB only one issue found: RTC INT pull-up 10K is reporting always LOW 1.0 Initial version with many Harware errors (MOSI routed to IO9, that needs to be pull-up in BOOT)"
Changed lines of the file:
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@@
     (effects (font (size 1.27 1.27)) (justify left bottom))
   )
-  (text "REV DESCRIPTION\n1.2 R12 RTC interrupt pull-up now changed to 4K7\n1.1 C3 working PCB only one issue found: RTC INT pull-up 10K is reporting always LOW\n1.0 Initial version with many Harware errors (MOSI routed to IO9, that needs to be pull-up in BOOT)"
-    (at 242.57 175.26 0)
+  (text "REV DESCRIPTION\n1.2 R12 RTC interrupt pull-up now changed to 4K7\n    Added R16 22Ω currrent limiter to charge RTC backup capacitors\n1.1 C3 working PCB only one issue found: RTC INT pull-up 10K is reporting always LOW\n1.0 Initial version with many Harware errors (MOSI routed to IO9, that needs to be pull-up in BOOT)"
+    (at 242.57 182.88 0)
     (effects (font (size 2 2)) (justify left bottom))
   )

Commit message: Optimize deepsleep for C3 version
Parts:
- added D6: 1N5819WS, Diode_SMD:D_SOD-323, symbol Diode:MBR0530
- J5: footprint footprint:MOLEX-I2C-532530470 -> footprint:MOLEX-I2C-Groove
Connections:
- net +5V: now also D6.2 (A); no longer C14.1, U3.3 (VI)
- new net: C14.1, D6.1 (K), U3.3 (VI)
Other:
- note added: "D6 prevents current leaking backwards when powered by 3.3V directly"
- note added: "REV DESCRIPTION 1.2 R12 RTC interrupt pull-up now changed to 4K7 Added R16 22Ω currrent limiter to charge RTC backup capacitors IMPORTANT: D6 to prevent LDO leak current backwards to UART (reducing in 4mA deepsleep) 1.1 C3 working PCB only one issue found: RTC INT pull-up 10K is reporting always LOW 1.0 Initial version with many Harware errors (MOSI routed to IO9, that needs to be pull-up in BOOT)"
- note removed: "REV DESCRIPTION 1.2 R12 RTC interrupt pull-up now changed to 4K7 Added R16 22Ω currrent limiter to charge RTC backup capacitors 1.1 C3 working PCB only one issue found: RTC INT pull-up 10K is reporting always LOW 1.0 Initial version with many Harware errors (MOSI routed to IO9, that needs to be pull-up in BOOT)"
